File: HLI-C_main/HLI-C_main.kicad_pcb (KiCad board)
At the start: 2 copper layers, 27.9 x 55 mm, 58 parts, among them CON1 USB_B, CON3 CR123A, CON4 Conn_02x05_Odd_Even, Q1 IRLML5103, U1 PIC24HJ64GP206-I_PT, U2 FM25V10-GTR, U3 FT232RL, U5 TPS7A0533PDBV, U6 LM3658SD, U7 TPS7A0533PDBV, U8 ATSHA204A-SSHDA-B, U9 24AA02-OT, Y1 Crystal_32KHz, Y2 Crystal_20MHz

Commit message: att
Parts:
- added R1: 0R, Resistor_SMD:R_0603_1608Metric_Pad0.98x0.95mm_HandSolder, F.Cu at (179.1, 41.4)
- moved C6 0.98 mm to (180.9, 41.5)
- moved U5 0.70 mm to (184.8, 40.8)
- moved D2 0.51 mm to (189.4, 40.7)
- renumbered R9 to R10, R10 to R11, R11 to R12, R12 to R13, R13 to R14, R1 to R2, R2 to R3, R3 to R4, R4 to R5, R5 to R6, R6 to R7, R7 to R8, R8 to R9
Connections:
- CON1 pad 6: 0 -> (no net)
- CON3 pad N: 0 -> (no net)
- CON4 pad 5: 0 -> GND
- Y1 pad 1: Net-(C23-Pad1) -> Net-(C22-Pad1)
- Y1 pad 2: Net-(C22-Pad1) -> Net-(C23-Pad1)
Routing:
- net Net-(C4-Pad1): track 32.6 -> 38.1 mm
- net +5VD: track 24.6 -> 22.6 mm, vias 3 -> 2
- net 0: track 57.1 -> 55.9 mm
