File: HLI-C_main/HLI-C_main.kicad_sch (KiCad schematic)
At the start: 57 parts, among them CON1 USB_B, CON3 CR123A, CON4 Conn_02x05_Odd_Even, Q1 IRLML5103, U1 PIC24HJ64GP206-I_PT, U2 FM25V10-GTR, U3 FT232RL, U5 TPS7A0533PDBV, U6 LM3658SD, U7 TPS7A0533PDBV, U8 ATSHA204A-SSHDA-B, U9 24AA02-OT, Y1 Crystal_32KHz, Y2 Crystal_20MHz

Commit message: att
Parts:
- added R1: 0R, Resistor_SMD:R_0603_1608Metric_Pad0.98x0.95mm_HandSolder, symbol Device:R
- CON4: value Conn_02x05_Odd_Even -> Conector_gravação
- renumbered R9 to R10, R10 to R11, R11 to R12, R12 to R13, R13 to R14, R1 to R2, R2 to R3, R3 to R4, R4 to R5, R5 to R6, R6 to R7, R7 to R8, R8 to R9
Connections:
- net +3V3: now also R1.1
- net at C4.1, U3.17 (3V3OUT), U3.4 (VCCIO): now also R1.2
Other:
- note added: "ALIMENTAÇÃO, COMUNICAÇÃO USB/SERIAL"
- note added: "CONECTOR PARA GRAVAÇÃO E COMUNICAÇÃO SERIAL"
- note added: "EEPROM"
- note added: "ENCRIPTAÇÃO"
- note added: "LEDS LOCKBITS"
- note added: "PIC e FRAM"
- note added: "PINO POWER"
- moved on the sheet: C1, C10, C11, C12, C13, C14, C15, C16, C17, C18, C19, C2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

Commit message: att
Parts:
- removed D1, D2, D3: SSA33L, Diode_SMD:D_SOD-123, symbol pspice:DIODE
- removed R1: 0R, Resistor_SMD:R_0603_1608Metric_Pad0.98x0.95mm_HandSolder, symbol Device:R
- added D1, D3: DSS14U, Diode_SMD:D_SOD-123, symbol Simulation_SPICE:DIODE
- added D2: S1D-13F, Diode_SMD:D_SMA, symbol Simulation_SPICE:DIODE
- added R15, R16: 470R, Resistor_SMD:R_0603_1608Metric_Pad0.98x0.95mm_HandSolder, symbol Device:R
- C11: value 100nF -> 1uF
- C20, C21: value 10pF -> 20pF
- C22, C23: value 7pF -> 12pF
- CON4: footprint Connector_PinSocket_1.27mm:PinSocket_2x05_P1.27mm_Vertical -> Connector_IDC:IDC-Header_2x05_P2.54mm_Vertical
Connections:
- net +5V: now also D1.1 (A), D3.1 (A)
- net +5VD: now also D1.2 (K)
- net 0: now also D2.1 (A)
- net RXA: now also R16.2; no longer U3.5 (RXD)
- net RXB: no longer U1.33 (U1TX/RF3)
- net TXA: now also R15.2; no longer U3.1 (TXD)
- net TXB: no longer U1.34 (U1RX/RF2)
- net VBAT: now also D2.2 (K)
- net K0: no longer names the net of U1.11 (RB5)
- net K1: no longer names the net of U1.12 (RB4)
- net K2: no longer names the net of U1.13 (RB3)
- net K3: no longer names the net of U1.14 (RB2)
- net K4: no longer names the net of U1.23 (RB10)
- net K5: no longer names the net of U1.24 (RB11)
- net K6: no longer names the net of U1.27 (RB12)
- net K7: no longer names the net of U1.28 (RB13)
- net K8: no longer names the net of U1.29 (RB14)
- net K9: no longer names the net of U1.30 (RB15)
- net KA: no longer names the net of U1.53 (RD5)
- net KB: no longer names the net of U1.52 (RD4)
- net KC: no longer names the net of U1.18 (RB7)
- net KD: no longer names the net of U1.21 (RB8)
- net KE: no longer names the net of U1.22 (RB9)
- new net: R15.1, U3.1 (TXD)
- new net: R16.1, U3.5 (RXD)
- no-connect marks 37 -> 54
Other:
- moved on the sheet: C2, C3
