File: HLI-M_3.1-FTD/HLI-M/HLI-M.kicad_pcb (KiCad board)
At the start: 2 copper layers, 125.2 x 86.1 mm, 122 parts, among them CON1 , CON2 USB_B, CON3 , CON4 Con_ADAPTER, CON5 Con_MULTLINKER, CON6 Conn_01x15, CON7 Conn_01x09, CON8 CR123A, Q1 DMP3068L-7, Q2 BC817, Q3 BC817, Q4 DMP2305, Q5 DMP2305, Q6 DMP2305, Q7 DMP2305, U1 PIC24HJ64GP206, U10 ULN2003, U11 ULN2003, U12 ULN2003, U2 FM25V10, U2-A DFN-8-1EP_6x5mm_P1.27mm_EP2x2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, U3 MAX3232, U4 ATSHA204A-SSHDA-B, U5 24AA02-OT, U5-A SOIC-8_3.9x4.9mm_P1.27mm, U6 LM3658SD, U7 TPS7A0533PDBV, U8 TPS7A0533PDBV, U9 FT232RL, Y1 Crystal_32KHz, Y2 Crystal_20MHz

Commit message: att
Parts:
- CON5: footprint Connector_IDC:IDC-Header_2x04_P2.54mm_Horizontal -> Connector_IDC:IDC-Header_2x05_P2.54mm_Horizontal
- R29: value 1K5 -> 1K8
- moved CON5 0.26 mm to (180.6, 76.3)
- moved R10 0.08 mm to (175.6, 87.1)
- moved R11 0.08 mm to (177.4, 87.1)
Connections:
- CON3 pad 20: 0 -> K_E
- CON5 pad 8: 0 -> EXTERN_D11
- CON8 pad N: 0 -> (no net)
- CON8 pad P: Net-(CON8-+) -> (no net)
- U1 pad 45: unconnected-(U1-RD11-Pad45) -> EXTERN_D11

Commit message: att
Parts:
- removed G1: LOGO, LOGO
- added G***: LOGO, LOGO, F.Cu at (93.7, 108.4)
Routing:
- net EXTERN_D11: track 0.00 -> 2.64 mm
- net 0: vias 47 -> 48
Other:
- board text added: "Made in China"
- board text removed: "Designed in Brazil. Made in China"
- board text removed: "SECURITY"

Commit message: att
Parts:
- added Q8: BC817, Package_TO_SOT_SMD:SOT-23, F.Cu at (170.7, 61.7)
- added R31: 22K, Resistor_SMD:R_0603_1608Metric_Pad0.98x0.95mm_HandSolder, F.Cu at (170.7, 58.5)
- added R32: 1K, Resistor_SMD:R_0603_1608Metric_Pad0.98x0.95mm_HandSolder, F.Cu at (167.2, 61.6)
- added R33: NC, Resistor_SMD:R_0603_1608Metric_Pad0.98x0.95mm_HandSolder, F.Cu at (170.8, 56.7)
Connections:
- CON3 pad 20: K_E -> 0
- CON3 pad 22: 0 -> K_E
- CON5 pad 10: 0 -> +12V
- CON5 pad 8: EXTERN_D11 -> HOOPER_
Routing:
- net EXTERN_D11: track 2.64 -> 54.1 mm, vias 0 -> 1
- net +12V: track 387.6 -> 393.1 mm, vias 5 -> 6
- net VBAT: track 224.8 -> 225.8 mm

Commit message: att
Parts:
- removed RV1: Varistor, Capacitor_SMD:C_0603_1608Metric_Pad1.08x0.95mm_HandSolder
- added D6: MMSZ5233B, Diode_SMD:D_SOD-123, F.Cu at (77.1, 45.2)
- F1: value Fuse -> 0.12A 30V; footprint Fuse:Fuse_1812_4532Metric -> Fuse:Fuse_1210_3225Metric
- moved R11 1.14 mm to (177.4, 86.0)
- moved R10 1.13 mm to (175.6, 86.0)
- moved F1 1.04 mm to (72.0, 45.5)
- moved R19 0.17 mm to (140.0, 57.2)
- turned Q8 to 0 degrees
Connections:
- CON8 pad N: (no net) -> 0
Routing:
- net HOOPER_: track 0.00 -> 46.8 mm, vias 0 -> 1
- net K_E: track 1.38 -> 21.1 mm, vias 1 -> 2
- net EXTERN_D11: track 54.1 -> 40.3 mm, vias 1 -> 2
- net +3V3: track 331.8 -> 343.0 mm
- net Net-(Q8-B): track 0.00 -> 3.59 mm
- net +12V: track 393.1 -> 390.3 mm
- net 0: track 63.2 -> 65.2 mm, vias 48 -> 50
- net +5V: track 238.8 -> 236.9 mm
- net Net-(CON1-Pin_1): track 18.0 -> 16.2 mm
- net RXA: track 88.7 -> 89.9 mm
- net PIN-CIN: track 4.49 -> 5.59 mm
- net EXTERN_D10: track 49.3 -> 50.2 mm
- net PGEC2: track 62.7 -> 61.8 mm
- net KB: track 35.2 -> 34.5 mm
- net KA: track 36.4 -> 35.7 mm
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
Commit message: atualizado 6/6 HLI-M
Parts:
- moved R14 0.83 mm to (154.4, 82.8), turned to 90 degrees
- moved D4 0.13 mm to (112.4, 65.5)
- moved R9 0.08 mm to (127.3, 87.1)
Routing:
- net +5VD: track 133.9 -> 168.9 mm, vias 5 -> 7
- net +3V3: track 343.0 -> 335.0 mm, vias 29 -> 30
- net TXA: track 94.6 -> 92.3 mm
- net +2V5: track 35.6 -> 37.4 mm
- net EXTERN_D10: track 50.2 -> 51.7 mm
- net PGED2: track 67.6 -> 66.2 mm
- net +5V: track 236.9 -> 237.8 mm
- net VBAT: track 226.2 -> 225.3 mm
- net +3.3VP: track 165.4 -> 164.5 mm
- net COUT: track 53.0 -> 53.7 mm
- net Net-(U1-VDDCORE): track 19.5 -> 20.1 mm
- net 0: track 65.2 -> 65.0 mm, vias 50 -> 49
