File: HLI-M_3.1-FTD/HLI-M/HLI-M.kicad_sch (KiCad schematic)
At the start: 123 parts, among them CON1 , CON2 USB_B, CON3 , CON4 Con_ADAPTER, CON5 Con_MULTLINKER, CON6 Conn_01x15, CON7 Conn_01x09, CON8 CR123A, Q1 DMP3068L-7, Q2 BC817, Q3 BC817, Q4 DMP2305, Q5 DMP2305, Q6 DMP2305, Q7 DMP2305, Q8 BC817, U1 PIC24HJ64GP206, U10 ULN2003, U11 ULN2003, U12 ULN2003, U2 FM25V10, U3 MAX3232, U4 ATSHA204A-SSHDA-B, U5 24AA02-OT, U6 LM3658SD, U7 TPS7A0533PDBV, U8 TPS7A0533PDBV, U9 FT232RL, Y1 Crystal_32KHz, Y2 Crystal_20MHz

Commit message: atualizado 6/6 HLI-M
Connections:
- no-connect marks 46 -> 34
Changed lines of the file:
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@@
   (junction (at 161.036 181.864) (diameter 0) (color 0 0 0 0)
   )
-  (no_connect (at 322.58 119.38))
   (no_connect (at 371.094 223.266))
-  (no_connect (at 83.566 150.114))
-  (no_connect (at 64.643 124.333))
-  (no_connect (at 329.184 87.503))
   (no_connect (at 430.784 224.79))
   (no_connect (at 118.11 273.558))
@@
   (no_connect (at 77.47 286.258))
   (no_connect (at 132.842 215.392))
-  (no_connect (at 470.662 113.538))
   (no_connect (at 286.258 72.39))
   (no_connect (at 118.11 291.338))
   (no_connect (at 326.898 82.55))
-  (no_connect (at 105.283 171.831))
-  (no_connect (at 52.959 66.675))
   (no_connect (at 350.774 225.806))
-  (no_connect (at 475.742 121.412))
   (no_connect (at 430.784 227.33))
   (no_connect (at 291.973 171.45))
@@
   (no_connect (at 371.094 225.806))
   (no_connect (at 350.774 228.346))
-  (no_connect (at 298.196 236.601))
   (no_connect (at 472.44 217.17))
-  (no_connect (at 277.241 286.258))
   (no_connect (at 77.47 281.178))
-  (no_connect (at 50.292 27.178))
   (no_connect (at 118.11 293.878))
   (no_connect (at 118.11 298.958))
@@
   (no_connect (at 451.358 152.4))
   (no_connect (at 451.358 154.94))
-  (no_connect (at 63.627 90.551))
   (no_connect (at 118.11 288.798))
   (no_connect (at 371.094 228.346))
@@
     (stroke (width 0) (type default))
   )
-  (wire (pts (xy 289.56 134.366) (xy 289.56 133.858))
+  (wire (pts (xy 289.56 134.239) (xy 289.56 133.858))
     (stroke (width 0) (type default))
   )
@@
     )
   )
-  (symbol (lib_id "pspice:0") (at 289.56 134.366 0) (mirror y) (unit 1)
+  (symbol (lib_id "pspice:0") (at 289.56 134.239 0) (mirror y) (unit 1)
     (in_bom yes) (on_board yes) (dnp no)
-    (property "Reference" "#GND0107" (at 289.56 136.906 0)
+    (property "Reference" "#GND0107" (at 289.56 136.779 0)
       (effects (font (size 1.27 1.27)) hide)
     )
-    (property "Value" "0" (at 289.56 132.1054 0)
+    (property "Value" "0" (at 289.56 131.9784 0)
       (effects (font (size 1.27 1.27)) hide)
     )
-    (property "Footprint" "" (at 289.56 134.366 0)
+    (property "Footprint" "" (at 289.56 134.239 0)
       (effects (font (size 1.27 1.27)) hide)
     )
-    (property "Datasheet" "~" (at 289.56 134.366 0)
+    (property "Datasheet" "~" (at 289.56 134.239 0)
       (effects (font (size 1.27 1.27)) hide)
     )
@@
   (symbol (lib_id "Device:C") (at 289.56 130.048 0) (unit 1)
     (in_bom yes) (on_board yes) (dnp no)
-    (property "Reference" "C21" (at 284.988 133.096 0)
+    (property "Reference" "C21" (at 284.353 132.715 0)
       (effects (font (size 1.27 1.27)) (justify left))
     )
-    (property "Value" "20pF" (at 290.068 133.096 0)
+    (property "Value" "20pF" (at 290.957 132.715 0)
       (effects (font (size 1.27 1.27)) (justify left))
     )
