File: HLI-C_main/HLI-C_2.0/HLI-C_main.kicad_sch (KiCad schematic)
At the start: 59 parts, among them CON1 USB_B, CON3 CR123A, CON4 Conector_gravação, Q1 IRLML5103, U1 PIC24HJ64GP206-I_PT, U2 FM25V10-GTR, U3 FT232RL, U5 STLQ020C33R, U6 LM3658SD, U7 STLQ020C33R, U8 ATSHA204A-SSHDA-B, U9 24AA02-OT, Y1 Crystal_32KHz, Y2 Crystal_20MHz

Commit message: HLI-C 2023: atualizado e revisado.
Parts:
- removed D1, D3: DSS14U, Diode_SMD:D_SOD-123, symbol Simulation_SPICE:DIODE
- removed D2: S1D-13F, Diode_SMD:D_SMA, symbol Simulation_SPICE:DIODE
- added D1, D2, D3: DSS14U, Diode_SMD:D_SOD-123, symbol Device:D
- Q1: value IRLML5103 -> DMP3068L-7
- R12: value 1K5 -> 1K8
- R4: value 10k -> 3.3k
- R5: value 10k -> 22k
- U5, U7: value STLQ020C33R -> TPS7A0533PDBV
- renumbered C23 to C22, C22 to C23
Connections:
- net GND is gone; now on net 0: CON4.5 (Pin_5)
- net +5V: now also D1.2 (A), D2.2 (A)
- net +5VD: now also D1.1 (K)
- net 0: now also U6.11 (DAP), D3.2 (A)
- net RXB: now also U1.33 (U1TX/RF3)
- net TXB: now also U1.34 (U1RX/RF2)
- net VBAT: now also D3.1 (K)
- net at C22.1, Y1.2: now also U1.48 (RC14); no longer U1.47 (RC13)
- net at C23.1, Y1.1: now also U1.47 (RC13); no longer U1.48 (RC14)
- net at C10.1, C9.1, Q1.2 (S)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: now also D2.1 (K)
- no-connect marks 54 -> 51
Other:
- note added: "CHIP ENCRIPTAÇÃO."
- note added: "CONECTOR PARA GRAVAÇÃO E COMUNICAÇÃO SERIAL."
- note added: "EEPROM."
- note added: "LEDS LOCKBITS."
- note added: "PROCESSADOR E FRAM."
- note removed: "CONECTOR PARA GRAVAÇÃO E COMUNICAÇÃO SERIAL"
- note removed: "EEPROM"
- note removed: "ENCRIPTAÇÃO"
- note removed: "LEDS LOCKBITS"
- note removed: "PIC e FRAM"
- note removed: "PINO POWER"
- company: (none) -> ORION GAMES.
- title: Projeto HLI-C -> Projeto HLI-C 2023
- moved on the sheet: C22, C23, R12, R13, R3, Y1
