File: HLI-C_main/HLI-C_2.0/HLI-C_main.kicad_pcb (KiCad board)
At the start: 2 copper layers, 33 x 72.2 mm, 60 parts, among them CON1 USB_B, CON3 CR123A, CON4 Conector_gravação, Q1 IRLML5103, U1 PIC24HJ64GP206-I_PT, U2 FM25V10-GTR, U3 FT232RL, U5 STLQ020C33R, U6 LM3658SD, U7 STLQ020C33R, U8 ATSHA204A-SSHDA-B, U9 24AA02-OT, Y1 Crystal_32KHz, Y2 Crystal_20MHz

Commit message: inicio alteracoes HLI-C
Parts:
- moved C5 19.3 mm to (204.1, 72.1)
- moved C9 19.1 mm to (203.9, 52.9)
- moved C8 8.23 mm to (207.0, 43.9)
- moved D2 5.87 mm to (203.8, 39.4), turned to 0 degrees
- moved C13 4.94 mm to (205.0, 43.9)
- moved R8 4.93 mm to (201.0, 43.9)
- moved C12 4.91 mm to (203.0, 43.9)
- moved Q1 0.32 mm to (204.3, 35.2), turned to -90 degrees
- moved C2 0.24 mm to (181.2, 23.6)
- moved C3 0.24 mm to (181.2, 21.3)
- moved C4 0.24 mm to (181.2, 19.0)
- moved C1 0.24 mm to (181.2, 25.9)
- moved U7 0.15 mm to (196.9, 34.3)
- turned RT1 to 0 degrees
Connections:
- CON4 pad 5: GND -> 0
- D3 pad 2: unconnected-(D3-Pad2) -> Net-(C7-Pad1)
Routing:
- net 0: track 13.1 -> 33.0 mm, vias 8 -> 12
- net Net-(C10-Pad1): track 43.7 -> 26.6 mm, vias 0 -> 2
- net +3V3: track 108.7 -> 125.0 mm, vias 0 -> 7
- net Net-(C7-Pad1): track 8.72 -> 24.3 mm, vias 0 -> 2
- net +5VD: track 61.8 -> 48.3 mm, vias 0 -> 4
- net Net-(U1-Pad5): track 14.5 -> 3.87 mm
- net Net-(C13-Pad1): track 37.0 -> 30.2 mm, vias 3 -> 2
- net Net-(R8-Pad2): track 20.4 -> 14.2 mm
- net Net-(CON3-Pad1): track 16.0 -> 11.7 mm
- net +5V: track 57.3 -> 60.7 mm, vias 0 -> 2
- net Net-(C18-Pad1): track 31.4 -> 29.1 mm
- net +3.3VP: track 96.1 -> 94.6 mm
- net Net-(C4-Pad1): track 27.6 -> 28.9 mm
- net TXA: track 17.1 -> 17.8 mm
- net LED2: track 7.42 -> 7.98 mm
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Other:
- board size 33 x 72.2 mm -> 33 x 73 mm

Commit message: circuito HLI-C finalizado, precisa de revisao
Parts:
- moved C22 1.74 mm to (180.5, 73.9)
- moved Y1 1.74 mm to (181.8, 69.0)
- moved C23 1.74 mm to (183.1, 73.9)
- moved C16 0.58 mm to (198.7, 74.0)
- moved LED2 0.58 mm to (187.3, 70.2)
- moved R10 0.58 mm to (191.2, 73.9)
- moved R11 0.58 mm to (189.3, 73.9)
- moved R15 0.58 mm to (187.3, 73.9)
- moved C17 0.58 mm to (196.8, 74.0)
- moved C18 0.58 mm to (194.9, 74.0)
- moved LED1 0.58 mm to (185.4, 70.1)
- moved R14 0.58 mm to (185.4, 73.8)
Connections:
- U1 pad 47: Net-(C23-Pad1) -> Net-(C22-Pad1)
- U1 pad 48: Net-(C22-Pad1) -> Net-(C23-Pad1)
Routing:
- net Net-(U1-Pad5): track 3.87 -> 14.6 mm
- net Net-(C22-Pad1): track 4.04 -> 13.8 mm
- net Net-(C23-Pad1): track 4.06 -> 12.1 mm
- net +3V3: track 125.0 -> 119.4 mm
- net Net-(C20-Pad1): track 3.35 -> 7.45 mm
- net 0: track 33.0 -> 36.2 mm, vias 12 -> 16
- net +3.3VP: track 94.6 -> 97.4 mm, vias 0 -> 2
- net Net-(C21-Pad1): track 6.09 -> 8.43 mm
- net PGED2: track 33.4 -> 31.8 mm
- net RESET: track 28.0 -> 29.4 mm, vias 0 -> 2
- net +5VD: track 48.3 -> 46.9 mm
- net Net-(U1-Pad6): track 18.5 -> 17.2 mm
- net Net-(C13-Pad1): track 30.2 -> 31.1 mm, vias 2 -> 0
- net Net-(LED1-Pad2): track 3.11 -> 2.39 mm
Other:
- board text added: "1"
- board text added: "17"
- board text added: "33"
- board text added: "49"

Commit message: HLI-C 2023: atualizado e revisado.
Parts:
- D2: value S1D-13F -> DSS14U; footprint Diode_SMD:D_SMA -> Diode_SMD:D_SOD-123
- Q1: value IRLML5103 -> DMP3068L-7
- R12: value 1K5 -> 1K8
- R4: value 10k -> 3.3k
- R5: value 10k -> 22k
- U5, U7: value STLQ020C33R -> TPS7A0533PDBV
- moved D3 17.4 mm to (204.1, 39.4)
- moved D2 17.2 mm to (203.8, 22.1)
- moved G1 10.8 mm to (192.7, 22.1)
- moved D1 0.09 mm to (203.8, 19.3), turned to 0 degrees
- renumbered C23 to C22, C22 to C23
Connections:
- C10 pad 1: Net-(C10-Pad1) -> Net-(D2-K)
- C7 pad 1: Net-(C7-Pad1) -> Net-(U6-USB_SEL)
- C9 pad 1: Net-(C10-Pad1) -> Net-(D2-K)
- CON3 pad P: Net-(CON3-Pad1) -> (no net)
- D1 pad 1: +5V -> +5VD
- D1 pad 2: +5VD -> +5V
- D2 pad 1: 0 -> Net-(D2-K)
- D2 pad 2: VBAT -> +5V
- D3 pad 1: +5V -> VBAT
- D3 pad 2: Net-(C7-Pad1) -> 0
- Q1 pad 2: Net-(C10-Pad1) -> Net-(D2-K)
- RT1 pad 1: Net-(CON3-Pad1) -> Net-(CON3-+)
- U1 pad 33: unconnected-(U1-Pad33) -> RXB
- U1 pad 34: unconnected-(U1-Pad34) -> TXB
- U6 pad 4: Net-(C7-Pad1) -> Net-(U6-USB_SEL)
- U7 pad 1: Net-(C10-Pad1) -> Net-(D2-K)
- U7 pad 3: Net-(C10-Pad1) -> Net-(D2-K)
Routing:
- net Net-(D2-K): track 0.00 -> 41.0 mm, vias 0 -> 4
- net RXB: track 0.00 -> 36.8 mm, vias 0 -> 1
- net TXB: track 0.00 -> 33.3 mm, vias 0 -> 1
- net Net-(C10-Pad1): track 26.6 -> 0.00 mm, vias 2 -> 0
- net Net-(C7-Pad1): track 24.3 -> 0.00 mm, vias 2 -> 0
- net Net-(CON3-Pad1): track 11.7 -> 0.00 mm, vias 1 -> 0
- net Net-(CON3-+): track 0.00 -> 11.7 mm, vias 0 -> 1
- net Net-(U6-USB_SEL): track 0.00 -> 8.72 mm
- net VBAT: track 85.1 -> 84.1 mm
- net +3V3: track 119.4 -> 120.1 mm
- net 0: track 36.2 -> 35.9 mm, vias 16 -> 17

Commit message: atualização serigrafia e conector bateria
Other:
- board text added: "Designed in Brazil. Made in China"
- board text added: "ORION.HLI-C 2023 REV A"

Commit message: att
Parts:
- removed G1: LOGO, LOGO
- added G***: LOGO, LOGO, B.Cu at (192.8, 22.2)
- moved C5 0.98 mm to (204.9, 71.6)
- moved C9 0.95 mm to (204.9, 53.1)
- moved C19 0.87 mm to (204.1, 64.3)
- moved C15 0.82 mm to (204.1, 60.2)
Routing:
- net +3V3: track 120.1 -> 121.1 mm
- net 0: track 35.9 -> 34.8 mm, vias 17 -> 18
- net Net-(U1-VDDCORE): track 28.9 -> 29.7 mm
- net +3.3VP: track 97.0 -> 97.6 mm
Other:
- board size 33 x 73 mm -> 34.2 x 73 mm
